Commit message: added camera topics to gazebo sim

File: src/ur5e_sim/urdf/camera.xacro (robot description, xacro)
@@ -1,78 +1,81 @@
 <?xml version="1.0"?>
 <robot xmlns:xacro="http://ros.org/wiki/xacro">
-    <material name="red">
-        <color rgba="1 0 0 1"/>
-    </material>
+  <material name="red">
+    <color rgba="1 0 0 1"/>
+  </material>
+  <!-- Macro: attach a depth camera to any parent link -->
+  <xacro:macro name="ur5e_depth_camera" params="parent_link *origin">
     <link name="camera_link">
-        <inertial>
-            <origin xyz="-0.00936000000 -0.00003000000 -0.00273000000" rpy="0 0 0"/>
-            <mass value="0.21970000000"/>
-            <inertia ixx="0.00000429247" ixy="0.00000000000" ixz="0.00000002565"
-                    iyy="0.00000008027" iyz="0.00000000000"
-                    izz="0.00000427339"/>
-        </inertial>
-        <visual>
-            <geometry>
-                <!-- <box size="0.01 0.03 0.03" /> -->
-                <mesh filename="package://ur5e_sim/meshes/sensors/camera/kinetic.stl"/>
-            </geometry>
-            <material name="red"/>
-        </visual>
-        <collision>
-            <geometry>
-                <mesh filename="package://ur5e_sim/meshes/sensors/camera/kinetic.dae"/>
-            </geometry>
-        </collision>
+      <inertial>
+        <origin xyz="-0.00936000000 -0.00003000000 -0.00273000000" rpy="0 0 0"/>
+        <mass value="0.21970000000"/>
+        <inertia ixx="0.00000429247" ixy="0.00000000000" ixz="0.00000002565"
+                 iyy="0.00000008027" iyz="0.00000000000"
+                 izz="0.00000427339"/>
+      </inertial>
+      <visual>
+        <geometry>
+          <!-- <box size="0.01 0.03 0.03" /> -->
+          <mesh filename="package://ur5e_sim/meshes/sensors/camera/kinetic.stl"/>
+        </geometry>
+        <material name="red"/>
+      </visual>
+      <collision>
+        <geometry>
+          <mesh filename="package://ur5e_sim/meshes/sensors/camera/kinetic.dae"/>
+        </geometry>
+      </collision>
     </link>
     <!-- frames in the center of the camera -->
     <joint name="camera_joint" type="fixed">
-        <parent link="base_link"/>
-        <child link="camera_link"/>
-        <origin xyz="0.5 0 1.2" rpy="0 1.57 0" />
+      <parent link="${parent_link}"/>
+      <child link="camera_link"/>
+      <!-- pose of camera relative to parent -->
+      <xacro:insert_block name="origin"/>
     </joint>
-    <link name="camera_optical_link"></link>
+    <link name="camera_optical_link"/>
     <joint name="camera_optical_joint" type="fixed">
-        <parent link="camera_link"/>
-        <child link="camera_optical_link"/>
-        <origin xyz="0 0 0" rpy="-1.57 0 -1.57" />
+      <parent link="camera_link"/>
+      <child link="camera_optical_link"/>
+      <origin xyz="0 0 0" rpy="-1.57 0 -1.57" />
     </joint>
     <gazebo reference="camera_link">
-        <visual>
-            <geometry>
-                <mesh>
-                    <uri>package://ur5e_sim/meshes/sensors/camera/kinetic.stl</uri>
-                </mesh>
-            </geometry>
-            <material>Gazebo/Red</material>
-        </visual>
-        <!-- <material>Gazebo/Red</material> -->
-        <sensor name="camera" type="depth">
-            <pose> 0 0 0 0 0 0 </pose>
-            <visualize>true</visualize>
-            <update_rate>10</update_rate>
-            <camera>
-                <horizontal_fov>1.089</horizontal_fov>
-                <image>
-                    <format>R8G8B8</format>
-                    <width>640</width>
-                    <height>480</height>
-                </image>
-                <clip>
-                    <near>0.05</near>
-                    <far>8</far>
-                </clip>
-            </camera>
-            <plugin name="camera_controller" filename="libgazebo_ros_camera.so" >
-                <frame_name>camera_optical_link</frame_name>
-            </plugin>
-        </sensor>
+      <visual>
+        <geometry>
+          <mesh>
+            <uri>package://ur5e_sim/meshes/sensors/camera/kinetic.stl</uri>
+          </mesh>
+        </geometry>
+        <material>Gazebo/Red</material>
+      </visual>
+      <sensor name="camera" type="depth">
+        <pose> 0 0 0 0 0 0 </pose>
+        <visualize>true</visualize>
+        <update_rate>10</update_rate>
+        <camera>
+          <horizontal_fov>1.089</horizontal_fov>
+          <image>
+            <format>R8G8B8</format>
+            <width>640</width>
+            <height>480</height>
+          </image>
+          <clip>
+            <near>0.05</near>
+            <far>8</far>
+          </clip>
+        </camera>
+        <plugin name="camera_controller" filename="libgazebo_ros_camera.so" >
+          <frame_name>camera_optical_link</frame_name>
+        </plugin>
+      </sensor>
     </gazebo>
     <gazebo reference="camera_link">
-        <visual>
-            <geometry>
-                <mesh filename="package://ur5e_sim/meshes/sensors/camera/kinetic.stl"/>
-            </geometry>
-            <material>Gazebo/Red</material>
-        </visual>
+      <visual>
+        <geometry>
+          <mesh filename="package://ur5e_sim/meshes/sensors/camera/kinetic.stl"/>
+        </geometry>
+        <material>Gazebo/Red</material>
+      </visual>
     </gazebo>
+  </xacro:macro>
 </robot>

File: src/ur5e_sim/urdf/ur5_camera_gripper.urdf.xacro (robot description, xacro)
@@ -141,4 +141,8 @@
   <xacro:arg name="use_fake_hardware" default="true" />
   <xacro:arg name="com_port" default="/dev/ttyUSB0" />
+   <!-- Example: mount camera on tool0 -->
+  <xacro:ur5e_depth_camera parent_link="tool0">
+    <origin xyz="0.0 0.0 0.15" rpy="0 0 0" />
+  </xacro:ur5e_depth_camera>
   <!-- Import macros -->
   <xacro:include filename="$(find ur5e_sim)/urdf/robotiq_gripper_macro.xacro" />

Commit message: Fixed the issue of the camera and gripper not showing up make sure you have these installed
  ros-humble-gazebo-ros-pkgs \

  ros-humble-gazebo-msgs \

  gazebo \

  libgazebo-dev \

  ros-humble-gazebo-ros2-control

  ros-humble-ros2-control ros-humble-ros2-controllers ros-humble-gazebo-ros2-control

File: src/ur5e_sim/urdf/camera.xacro (robot description, xacro)
@@ -17,5 +17,5 @@
         <geometry>
           <!-- <box size="0.01 0.03 0.03" /> -->
-          <mesh filename="package://ur5e_sim/meshes/sensors/camera/kinetic.stl"/>
+          <mesh filename="file://${URYT}/meshes/sensors/camera/kinetic.stl"/>
         </geometry>
         <material name="red"/>
@@ -23,5 +23,5 @@
       <collision>
         <geometry>
-          <mesh filename="package://ur5e_sim/meshes/sensors/camera/kinetic.dae"/>
+          <mesh filename="file://${URYT}/meshes/sensors/camera/kinetic.dae"/>
         </geometry>
       </collision>
@@ -73,5 +73,5 @@
       <visual>
         <geometry>
-          <mesh filename="package://ur5e_sim/meshes/sensors/camera/kinetic.stl"/>
+          <mesh filename="file://${URYT}/meshes/sensors/camera/kinetic.stl"/>
         </geometry>
         <material>Gazebo/Red</material>

File: src/ur5e_sim/urdf/robotiq_gripper_macro.xacro (robot description, xacro)
@@ -43,10 +43,10 @@
             <visual>
                 <geometry>
-                    <mesh filename="package://robotiq_description/meshes/visual/2f_85/robotiq_base.dae" />
-                </geometry>
-            </visual>
-            <collision>
-                <geometry>
-                    <mesh filename="package://robotiq_description/meshes/collision/2f_85/robotiq_base.stl" />
+                    <mesh filename="file://${ROBI}/meshes/visual/2f_85/robotiq_base.dae"/>
+                </geometry>
+            </visual>
+            <collision>
+                <geometry>
+                    <mesh filename="file://${ROBI}/meshes/collision/2f_85/robotiq_base.stl"/>
                 </geometry>
             </collision>
@@ -60,10 +60,10 @@
             <visual>
                 <geometry>
-                    <mesh filename="package://robotiq_description/meshes/visual/2f_85/left_knuckle.dae" />
-                </geometry>
-            </visual>
-            <collision>
-                <geometry>
-                    <mesh filename="package://robotiq_description/meshes/collision/2f_85/left_knuckle.stl" />
+                    <mesh filename="file://${ROBI}/meshes/visual/2f_85/left_knuckle.dae" />
+                </geometry>
+            </visual>
+            <collision>
+                <geometry>
+                    <mesh filename="file://${ROBI}/meshes/collision/2f_85/left_knuckle.stl" />
                 </geometry>
             </collision>
@@ -77,10 +77,10 @@
             <visual>
                 <geometry>
-                    <mesh filename="package://robotiq_description/meshes/visual/2f_85/right_knuckle.dae" />
-                </geometry>
-            </visual>
-            <collision>
-                <geometry>
-                    <mesh filename="package://robotiq_description/meshes/collision/2f_85/right_knuckle.stl" />
+                    <mesh filename="file://${ROBI}/meshes/visual/2f_85/right_knuckle.dae" />
+                </geometry>
+            </visual>
+            <collision>
+                <geometry>
+                    <mesh filename="file://${ROBI}/meshes/collision/2f_85/right_knuckle.stl" />
                 </geometry>
             </collision>
@@ -94,10 +94,10 @@
             <visual>
                 <geometry>
-                    <mesh filename="package://robotiq_description/meshes/visual/2f_85/left_finger.dae" />
-                </geometry>
-            </visual>
-            <collision>
-                <geometry>
-                    <mesh filename="package://robotiq_description/meshes/collision/2f_85/left_finger.stl" />
+                    <mesh filename="file://${ROBI}/meshes/visual/2f_85/left_finger.dae" />
+                </geometry>
+            </visual>
+            <collision>
+                <geometry>
+                    <mesh filename="file://${ROBI}/meshes/collision/2f_85/left_finger.stl" />
                 </geometry>
             </collision>
@@ -111,10 +111,10 @@
             <visual>
                 <geometry>
-                    <mesh filename="package://robotiq_description/meshes/visual/2f_85/right_finger.dae" />
-                </geometry>
-            </visual>
-            <collision>
-                <geometry>
-                    <mesh filename="package://robotiq_description/meshes/collision/2f_85/right_finger.stl" />
+                    <mesh filename="file://${ROBI}/meshes/visual/2f_85/right_finger.dae" />
+                </geometry>
+            </visual>
+            <collision>
+                <geometry>
+                    <mesh filename="file://${ROBI}/meshes/collision/2f_85/right_finger.stl" />
                 </geometry>
             </collision>
@@ -128,10 +128,10 @@
             <visual>
                 <geometry>
-                    <mesh filename="package://robotiq_description/meshes/visual/2f_85/left_inner_knuckle.dae" />
-                </geometry>
-            </visual>
-            <collision>
-                <geometry>
-                    <mesh filename="package://robotiq_description/meshes/collision/2f_85/left_inner_knuckle.stl" />
+                    <mesh filename="file://${ROBI}/meshes/visual/2f_85/left_inner_knuckle.dae" />
+                </geometry>
+            </visual>
+            <collision>
+                <geometry>
+                    <mesh filename="file://${ROBI}/meshes/collision/2f_85/left_inner_knuckle.stl" />
                 </geometry>
             </collision>
@@ -145,10 +145,10 @@
             <visual>
                 <geometry>
-                    <mesh filename="package://robotiq_description/meshes/visual/2f_85/right_inner_knuckle.dae" />
-                </geometry>
-            </visual>
-            <collision>
-                <geometry>
-                    <mesh filename="package://robotiq_description/meshes/collision/2f_85/right_inner_knuckle.stl" />
+                    <mesh filename="file://${ROBI}/meshes/visual/2f_85/right_inner_knuckle.dae" />
+                </geometry>
+            </visual>
+            <collision>
+                <geometry>
+                    <mesh filename="file://${ROBI}/meshes/collision/2f_85/right_inner_knuckle.stl" />
                 </geometry>
             </collision>
@@ -162,10 +162,10 @@
             <visual>
                 <geometry>
-                    <mesh filename="package://robotiq_description/meshes/visual/2f_85/left_finger_tip.dae" />
-                </geometry>
-            </visual>
-            <collision>
-                <geometry>
-                    <mesh filename="package://robotiq_description/meshes/collision/2f_85/left_finger_tip.stl" />
+                    <mesh filename="file://${ROBI}  /meshes/visual/2f_85/left_finger_tip.dae" />
+                </geometry>
+            </visual>
+            <collision>
+                <geometry>
+                    <mesh filename="file://${ROBI}/meshes/collision/2f_85/left_finger_tip.stl" />
                 </geometry>
                 <surface>
@@ -197,10 +197,10 @@
             <visual>
                 <geometry>
-                    <mesh filename="package://robotiq_description/meshes/visual/2f_85/right_finger_tip.dae" />
-                </geometry>
-            </visual>
-            <collision>
-                <geometry>
-                    <mesh filename="package://robotiq_description/meshes/collision/2f_85/right_finger_tip.stl" />
+                    <mesh filename="file://${ROBI}/meshes/visual/2f_85/right_finger_tip.dae" />
+                </geometry>
+            </visual>
+            <collision>
+                <geometry>
+                    <mesh filename="file://${ROBI}/meshes/collision/2f_85/right_finger_tip.stl" />
                 </geometry>
                 <surface>

File: src/ur5e_sim/urdf/ur5_camera_gripper.urdf.xacro (robot description, xacro)
@@ -4,4 +4,6 @@
    <xacro:arg name="name" default="ur"/>
    <!-- import main macro -->
+   <xacro:property name="URYT" value="$(find ur5e_sim)"/>
+   <xacro:property name="ROBI" value="$(find robotiq_description)"/>
    <xacro:include filename="$(find ur5e_sim)/urdf/camera.xacro"/>
    <xacro:include filename="$(find ur5e_sim)/urdf/ur5_macro.xacro"/>
