Commit message: Changed the order joint_states is recieved, moved camera to wrist_3_link changed image_saver to save to my path instead of the og one made the model load from checkpoint instead of huggingface

File: src/ur5e_sim/urdf/ur5_camera_gripper.urdf.xacro (robot description, xacro)
@@ -143,7 +143,7 @@
   <xacro:arg name="use_fake_hardware" default="true" />
   <xacro:arg name="com_port" default="/dev/ttyUSB0" />
-   <!-- Example: mount camera on tool0 -->
-  <xacro:ur5e_depth_camera parent_link="tool0">
-    <origin xyz="0.0 0.0 0.15" rpy="0 0 0" />
+   <!-- Example: mount camera on wrist_3_link -->
+  <xacro:ur5e_depth_camera parent_link="wrist_3_link">
+    <origin xyz="0.0 -0.06 -0.027" rpy="0 -1.6 1.6" />
   </xacro:ur5e_depth_camera>
   <!-- Import macros -->

Commit message: Changed the home position for the arm changed the initial position of the red block does not move now, not sure if its because it believes its finished

File: src/ur5e_sim/urdf/ur5_camera_gripper.urdf.xacro (robot description, xacro)
@@ -145,5 +145,5 @@
    <!-- Example: mount camera on wrist_3_link -->
   <xacro:ur5e_depth_camera parent_link="wrist_3_link">
-    <origin xyz="0.0 -0.06 -0.027" rpy="0 -1.6 1.6" />
+    <origin xyz="0 -0.059 -0.035" rpy="0 -1.6 1.6" />
   </xacro:ur5e_depth_camera>
   <!-- Import macros -->

Commit message: Added rdt_scripts/ back

File: src/ur5e_sim/urdf/ur5_camera_gripper.urdf.xacro (robot description, xacro)
@@ -145,6 +145,11 @@
    <!-- Example: mount camera on wrist_3_link -->
   <xacro:ur5e_depth_camera parent_link="wrist_3_link">
-    <origin xyz="0 -0.059 -0.035" rpy="0 -1.6 1.6" />
+    <origin xyz="0 -0.063 -0.022" rpy="0 -1.6 1.6" />
   </xacro:ur5e_depth_camera>
+<!--
+  <xacro:ur5e_depth_camera parent_link="world" id="high_cam">
+    <origin xyz="0 0.059 4" rpy="0 1.6 -1.6" />
+  </xacro:ur5e_depth_camera>
+  -->
   <!-- Import macros -->
   <xacro:include filename="$(find ur5e_sim)/urdf/robotiq_gripper_macro.xacro" />
